File: kicad/Leverless_controller_v2/with_usb_wired_v1.kicad_pcb (KiCad board)
At the start: 2 copper layers, 224 x 139 mm, 22 parts

Commit message: Add files via upload
Parts:
- S1, S10, S11, S12, S13, S14, S2, S3, S4, S5, S6, S7, S8, S9: footprint Button_Switch_Keyboard:SW_Gateron_LowProfile_HotSwap_PTH_footprint -> Library:SW_Gateron_LowProfile_HotSwap_PTH_footprint
Other:
- outline, holes or cut-outs redrawn

Commit message: editing kicad file
Parts:
- S1, S10, S11, S12, S13, S14, S2, S3, S4, S5, S6, S7, S8, S9: footprint Library:SW_Gateron_LowProfile_HotSwap_PTH_footprint -> Button_Switch_Keyboard:SW_Gateron_LowProfile_HotSwap_PTH_footprint
- moved S6 5.10 mm to (230.0, 136.0)
- moved REF** 3.64 mm to (330.0, 150.5)
- moved S5 2.92 mm to (225.5, 178.5)
- moved S1 2.69 mm to (143.5, 142.0)
- moved S7 2.55 mm to (254.5, 166.5)
- moved S8 1.12 mm to (259.5, 133.0)
- moved S9 1.00 mm to (284.0, 163.0)
- moved S11 0.71 mm to (313.5, 163.5)
Routing:
- net p0: track 64.3 -> 61.2 mm
- net k0: track 97.7 -> 99.6 mm
- net k3: track 158.2 -> 159.7 mm
- net p1: track 82.5 -> 83.9 mm
- net k1: track 110.0 -> 110.5 mm
Other:
- board size 224 x 139 mm -> 227 x 141 mm
